Commit message: Laboratory #3

File: urdf/robot.xacro (robot description, xacro)
@@ -8,5 +8,5 @@
 	<!-- Invoke the macro to define the Hokuyo LIDAR. -->
 	<xacro:VLP-16 parent = "base" name = "laser_horiz" topic = "laser_horiz/packets" hz = "10" samples = "440" gpu = "false" >
-		< origin xyz = "0.2325416305773505 -0.0001380069427607134 1.920122926231907" rpy = "-0.0012068 0.114646 -0.0015308" />
+		<origin xyz = "0.2325416305773505 -0.0001380069427607134 1.920122926231907" rpy = "-0.0012068 0.114646 -0.0015308" />
 	</xacro:VLP-16>
   <link name="base">
