Commit message: New file for HW3

File: urdf/base_robot.xacro (robot description, xacro)
@@ -15,12 +15,12 @@
 	<link name="imu">
 		<visual>
-		<geometry>
-		<sphere radius="0.1" />
-		</geometry>
+			<geometry>
+				<sphere radius="0.1" />
+			</geometry>
 		</visual>
 		<collision>
-		<geometry>
-		<sphere radius="0.1" />
-		</geometry>
+			<geometry>
+				<sphere radius="0.1" />
+			</geometry>
 		</collision>
 	</link>
